File: INVBackMeasurement.kicad_pcb (KiCad board)
At the start: 2 copper layers, 90 parts, among them IC1 TC1014-3.0VCT713, IC2 HCPL-181-000E, IC3 HCPL-181-000E, IC4 HCPL-181-000E, IC5 HCPL-181-000E, IC6 HCPL-181-000E, IC7 HCPL-181-000E, J1 PV(max600VDC), J10 ZCD, J2 AN_IN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

Commit message: the new one 2/10/2019
Parts:
- moved J10 200.8 mm to (33.8, 89.8), turned to 90 degrees
- moved IC7 192.4 mm to (35.0, 82.8), turned to 270 degrees
- moved J7 192.3 mm to (43.1, 89.8), turned to 90 degrees
- moved R29 186.5 mm to (35.4, 77.3), turned to 0 degrees
- moved R30 186.1 mm to (28.4, 34.5), turned to 90 degrees
- moved J9 184.3 mm to (52.4, 89.8), turned to 90 degrees
- moved R28 184.0 mm to (35.4, 74.8), turned to 0 degrees
- moved IC5 183.5 mm to (44.4, 82.8), turned to 270 degrees
- moved D7 181.9 mm to (38.4, 75.7), turned to 90 degrees
- moved R31 181.1 mm to (32.4, 34.5), turned to 270 degrees
- moved R26 177.4 mm to (44.7, 77.3), turned to 0 degrees
- moved J8 177.1 mm to (61.8, 89.8), turned to 90 degrees
- moved R32 176.0 mm to (36.4, 34.5), turned to 90 degrees
- moved IC4 175.3 mm to (53.7, 82.8), turned to 270 degrees
- moved R22 174.8 mm to (44.7, 74.8), turned to 0 degrees
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Routing:
- net GNDD: track 0.00 -> 54.5 mm, vias 0 -> 6
- net Net-(IC7-Pad4): track 0.00 -> 3.92 mm
- net Net-(IC7-Pad3): track 0.00 -> 3.92 mm
- net Net-(IC5-Pad4): track 0.00 -> 3.92 mm
- net Net-(IC5-Pad3): track 0.00 -> 3.92 mm
- net Net-(IC4-Pad4): track 0.00 -> 3.92 mm
- net Net-(IC4-Pad3): track 0.00 -> 3.92 mm
- net Net-(IC3-Pad4): track 0.00 -> 3.92 mm
- net Net-(IC3-Pad3): track 0.00 -> 3.92 mm
- net /ZCD: track 0.00 -> 2.50 mm
- net /PWD: track 0.00 -> 2.50 mm
- net /EVENT2: track 0.00 -> 2.50 mm
- net /EVENT1: track 0.00 -> 2.50 mm
- net Net-(IC7-Pad1): track 0.00 -> 2.42 mm
- net Net-(IC5-Pad1): track 0.00 -> 2.42 mm
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- added copper zone on F.Cu, net GNDD
Other:
- board outline added: 137.2 x 81 mm

Commit message: the new one
Parts:
- added J11: Screw_Terminal_01x02, TerminalBlock:TerminalBlock_Wuerth_691311400102_P7.62mm, F.Cu at (173.8, 38.4)
- added R33: CSNL2512FT2L00, InvertorMeasurement_kicad:ShuntMF0.0002Ohm2512, F.Cu at (139.7, 57.4)
- R12: value 2m -> 2.49R; footprint InvertorMeasurement_kicad:ShuntMF0.0002Ohm2512 -> Resistor_SMD:R_0805_2012Metric
- moved R9 83.2 mm to (167.7, 91.9)
- moved L3 79.2 mm to (174.1, 66.3), turned to 0 degrees
- moved C3 79.1 mm to (114.4, 128.0), turned to 180 degrees
- moved R11 77.8 mm to (167.6, 80.0), turned to 270 degrees
- moved R5 73.6 mm to (154.7, 93.3), turned to 0 degrees
- moved D6 71.9 mm to (98.6, 75.1), turned to 90 degrees
- moved R23 70.6 mm to (98.6, 70.2), turned to 270 degrees
- moved L1 69.7 mm to (169.7, 57.4), turned to 90 degrees
- moved PS1 66.2 mm to (154.8, 113.8)
- moved R27 64.3 mm to (94.6, 70.2), turned to 270 degrees
- moved C9 63.7 mm to (144.2, 91.9)
- moved R6 62.7 mm to (153.3, 82.4), turned to 270 degrees
- moved C5 60.2 mm to (96.0, 94.7), turned to 90 degrees
- moved C18 58.5 mm to (44.7, 95.7), turned to 0 degrees
- moved IC2 57.4 mm to (87.3, 92.8)
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Connections:
- L1 pad 2: Net-(L1-Pad2) -> /AC\L_OUT
- L2 pad 2: Net-(L2-Pad2) -> /AC\L
- R12 pad 1: /AC\L -> Net-(L1-Pad1)
- R12 pad 2: Net-(L2-Pad2) -> Net-(L2-Pad1)
Routing:
- net GNDD: track 54.5 -> 342.3 mm, vias 6 -> 9
- net /AC\N: track 0.00 -> 150.3 mm
- net /AC\L: track 0.00 -> 110.1 mm, vias 0 -> 2
- net Net-(C10-Pad1): track 0.00 -> 101.6 mm, vias 0 -> 2
- net Net-(C13-Pad1): track 0.00 -> 87.1 mm, vias 0 -> 4
- net Net-(C9-Pad2): track 0.00 -> 79.7 mm
- net Net-(L1-Pad1): track 0.00 -> 65.3 mm
- net GNDPWR: track 0.00 -> 63.0 mm
- net Net-(L2-Pad1): track 0.00 -> 62.5 mm
- net Net-(J1-Pad2): track 0.00 -> 60.0 mm, vias 0 -> 2
- net /STRINGDC+: track 0.00 -> 59.4 mm
- net /VOLTDC: track 0.00 -> 46.8 mm
- net Net-(C1-Pad1): track 0.00 -> 42.8 mm
- net Net-(C2-Pad1): track 0.00 -> 33.4 mm
- net Net-(C15-Pad1): track 0.00 -> 32.9 mm
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- added copper zone on F.Cu, net /3.3VDC
- added copper zone on F.Cu, net /AC\L
- added copper zone on F.Cu, net /AC\L_OUT
- added copper zone on F.Cu, net /AC\N
- added copper zone on B.Cu, net GNDD
- added copper zone on F.Cu, net GNDPWR
- added copper zone on F.Cu, net Net-(J1-Pad2)
- removed copper zone on F.Cu, net GNDD
Other:
- board outline removed

Commit message: 3/10/2019
Parts:
- moved C15 4.07 mm to (48.8, 79.0)
- moved C18 4.07 mm to (48.8, 95.9)
- moved Y2 4.07 mm to (47.9, 84.9)
Connections:
- R22 pad 1: /PWD -> /PWM
- R26 pad 1: /PWD -> /PWM
Routing:
- net GNDPWR: track 63.0 -> 394.9 mm, vias 0 -> 10
- net /AVDD: track 9.69 -> 214.4 mm, vias 0 -> 8
- net Net-(J2-Pad1): track 0.00 -> 184.5 mm, vias 0 -> 1
- net /3.3VDC: track 29.1 -> 151.3 mm, vias 2 -> 11
- net /GPD: track 0.00 -> 84.8 mm, vias 0 -> 3
- net /ZCD: track 4.00 -> 80.3 mm, vias 0 -> 2
- net /PWM: track 0.00 -> 58.8 mm, vias 0 -> 2
- net /GPC: track 0.00 -> 58.0 mm, vias 0 -> 1
- net /EVENT2: track 4.00 -> 54.7 mm, vias 0 -> 2
- net /EVENT1: track 4.00 -> 54.3 mm, vias 0 -> 3
- net GNDD: track 342.3 -> 385.4 mm, vias 9 -> 17
- net /PWD: track 4.00 -> 0.00 mm
- net Net-(IC7-Pad1): track 0.00 -> 3.43 mm
- net Net-(C18-Pad1): track 31.3 -> 29.9 mm
- net Net-(C15-Pad1): track 32.9 -> 32.0 mm
Other:
- board outline added: 186.7 x 119.6 mm
