File: INVBackMeasurement.sch (KiCad schematic (older format))
At the start: 82 parts, among them IC1 TC1014-3.0VCT713, IC2 HCPL-181-000E, IC3 HCPL-181-000E, IC4 HCPL-181-000E, IC5 HCPL-181-000E, IC6 HCPL-181-000E, J1 PV(DC), J2 AN_IN, J3 STRINGTOINVERTER, J4 SPI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

Commit message: 29/9/2019 9:52 PM
Parts:
- added D7: LED, LED_SMD:LED_0805_2012Metric, symbol Device:LED
- added IC7: HCPL-181-000E, InvertorMeasurement_kicad:HCPL-181-000E, symbol UImeasurement:HCPL-181-000E
- added J10: ZCD, Connector_PinHeader_2.54mm:PinHeader_1x02_P2.54mm_Vertical, symbol Connector:Conn_01x02_Male
- added R28, R29: 1K, symbol Device:R
- added R30: 1M, Resistor_SMD:R_1206_3216Metric, symbol Device:R
- added R31, R32: 47K, Resistor_SMD:R_1206_3216Metric, symbol Device:R
- C1, C11, C14, C15, C18, C2, C21, C6, C7, C8: footprint (none) -> Capacitor_SMD:C_0805_2012Metric
- C10, C12, C13, C16, C17, C19, C20, C3, C4, C5, C9: footprint (none) -> Capacitor_SMD:C_1206_3216Metric
- C22: footprint (none) -> Capacitor_SMD:C_1210_3225Metric
- D1, D2, D3, D4, D5, D6: footprint (none) -> LED_SMD:LED_0805_2012Metric
- IC1: footprint SOT95P270X145-5N -> InvertorMeasurement_kicad:TC1014-3.0V
- IC2, IC3, IC4, IC5, IC6: footprint SOP254P675X240-4N -> InvertorMeasurement_kicad:HCPL-181-000E
- J1: value PV(DC) -> PV(max600VDC); footprint (none) -> TerminalBlock:TerminalBlock_Wuerth_691311400102_P7.62mm
- J2: footprint (none) -> Connector_PinHeader_2.54mm:PinHeader_1x01_P2.54mm_Vertical
- J3, J5: footprint (none) -> TerminalBlock:TerminalBlock_Wuerth_691311400102_P7.62mm
- J4: footprint (none) -> Connector_PinHeader_2.54mm:PinHeader_1x04_P2.54mm_Vertical
- J6: footprint (none) -> Connector_PinHeader_2.54mm:PinHeader_1x05_P2.54mm_Vertical
- J7: value Conn_01x02_Female -> PWD; footprint (none) -> Connector_PinSocket_2.54mm:PinSocket_1x02_P2.54mm_Vertical
- J8: value Conn_01x02_Male -> EVENT1; footprint (none) -> Connector_PinHeader_2.54mm:PinHeader_1x02_P2.54mm_Vertical
- J9: value Conn_01x02_Male -> EVENT2; footprint (none) -> Connector_PinHeader_2.54mm:PinHeader_1x02_P2.54mm_Vertical
- L1, L2, L3, L5: footprint (none) -> Inductor_SMD:L_1206_3216Metric
- L4: footprint (none) -> Inductor_SMD:L_0805_2012Metric
- R1, R11, R4, R5, R6, R7, R8, R9: footprint (none) -> Resistor_SMD:R_1206_3216Metric
- R10: footprint (none) -> Resistor_SMD:R_0805_2012Metric
- R12: footprint (none) -> InvertorMeasurement_kicad:ShuntMF0.0002Ohm2512
- R2, R3: value R -> 3.3K; footprint (none) -> Resistor_SMD:R_1206_3216Metric
- R20, R21, R22, R23, R24, R25, R26, R27: value R -> 1K
- U1: footprint (none) -> InvertorMeasurement_kicad:MCP39F511
- U2: footprint digikey-footprints:SOIC-8_W3.9mm -> InvertorMeasurement_kicad:ACS712ELCTR-20A-T
- U3: footprint (none) -> InvertorMeasurement_kicad:dsPIC33CK256MP502
- Y1, Y2: footprint (none) -> Crystal:Crystal_HC49-U_Vertical
Connections:
- net GNDD: now also D7.1 (K), IC7.2 (K)
- net GNDPWR: now also R2.2; no longer R3.2
- net RX: now also IC2.4 (C); no longer R14.1
- net TXMCU: now also R14.1; no longer IC2.1 (A)
- net VOLTDC: now also R32.2; no longer R2.2
- net ZCD: now also R28.1, R29.1
- net at U2.1 (IP+), U2.2 (IP+): no longer J1.2 (Pin_2), R2.1
- net at R14.2: now also IC2.1 (A); no longer IC2.4 (C)
- new net: J1.2 (Pin_2), R30.1
- new net: R2.1, R3.2
- new net: IC7.1 (A), R29.2
- new net: IC7.3 (E), J10.1 (Pin_1)
- new net: IC7.4 (C), J10.2 (Pin_2)
- new net: D7.2 (A), R28.2
- new net: R31.2, R32.1
- new net: R30.2, R31.1
Other:
- moved on the sheet: D2, J1, PS1, R15, R2, R3

Commit message: the new one 1/10/2019
Parts:
- R13, R14, R15, R16, R17, R18, R19, R20, R21, R22, R23, R24, R25, R26, R27, R28, R29: footprint (none) -> Resistor_SMD:R_0805_2012Metric
- SW1: footprint (none) -> Button_Switch_THT:SW_PUSH_6mm_H5mm
Connections:
- net AC\L: now also J5.2 (Pin_2); no longer J5.1 (Pin_1)
- net AC\N: now also J5.1 (Pin_1); no longer J5.2 (Pin_2)
- net at U2.1 (IP+), U2.2 (IP+): now also J1.2 (Pin_2), R30.1
- net at IC5.3 (E): now also J7.1 (Pin_1); no longer J7.2 (Pin_2)
- net at IC5.4 (C): now also J7.2 (Pin_2); no longer J7.1 (Pin_1)
Changed lines of the file:
@@
 F 0 "SW1" H 9200 4885 50  0000 C CNN
 F 1 "RESET" H 9200 4794 50  0000 C CNN
-F 2 "" H 9200 4800 50  0001 C CNN
+F 2 "Button_Switch_THT:SW_PUSH_6mm_H5mm" H 9200 4800 50  0001 C CNN
 F 3 "~" H 9200 4800 50  0001 C CNN
 	1    9200 4600
@@
 F 0 "R17" H 8820 4346 50  0000 L CNN
 F 1 "R" H 8820 4255 50  0000 L CNN
-F 2 "" V 8680 4300 50  0001 C CNN
+F 2 "Resistor_SMD:R_0805_2012Metric" V 8680 4300 50  0001 C CNN
 F 3 "~" H 8750 4300 50  0001 C CNN
 	1    8750 4300
@@
 Connection ~ 2200 1700
 Wire Wire Line
-	2200 1400 2500 1400
-Wire Wire Line
 	2200 1500 2500 1500
-Wire Wire Line
-	2200 1150 2550 1150
-Wire Wire Line
-	2200 1400 2200 1500
 Wire Wire Line
 	3300 1500 4300 1500
@@
 F 0 "R20" H 9470 796 50  0000 L CNN
 F 1 "1K" H 9470 705 50  0000 L CNN
-F 2 "" V 9330 750 50  0001 C CNN
+F 2 "Resistor_SMD:R_0805_2012Metric" V 9330 750 50  0001 C CNN
 F 3 "~" H 9400 750 50  0001 C CNN
 	1    9400 750
@@
 F 0 "R24" H 9870 796 50  0000 L CNN
 F 1 "1K" H 9870 705 50  0000 L CNN
-F 2 "" V 9730 750 50  0001 C CNN
+F 2 "Resistor_SMD:R_0805_2012Metric" V 9730 750 50  0001 C CNN
 F 3 "~" H 9800 750 50  0001 C CNN
 	1    9800 750
@@
 F 0 "R21" H 9470 1696 50  0000 L CNN
 F 1 "1K" H 9470 1605 50  0000 L CNN
-F 2 "" V 9330 1650 50  0001 C CNN
+F 2 "Resistor_SMD:R_0805_2012Metric" V 9330 1650 50  0001 C CNN
 F 3 "~" H 9400 1650 50  0001 C CNN
 	1    9400 1650
@@
 F 0 "R25" H 9870 1696 50  0000 L CNN
 F 1 "1K" H 9870 1605 50  0000 L CNN
-F 2 "" V 9730 1650 50  0001 C CNN
+F 2 "Resistor_SMD:R_0805_2012Metric" V 9730 1650 50  0001 C CNN
 F 3 "~" H 9800 1650 50  0001 C CNN
 	1    9800 1650
@@
 F 0 "R22" H 9470 2546 50  0000 L CNN
 F 1 "1K" H 9470 2455 50  0000 L CNN
-F 2 "" V 9330 2500 50  0001 C CNN
+F 2 "Resistor_SMD:R_0805_2012Metric" V 9330 2500 50  0001 C CNN
 F 3 "~" H 9400 2500 50  0001 C CNN
 	1    9400 2500
@@
 F 0 "R26" H 9870 2546 50  0000 L CNN
 F 1 "1K" H 9870 2455 50  0000 L CNN
-F 2 "" V 9730 2500 50  0001 C CNN
+F 2 "Resistor_SMD:R_0805_2012Metric" V 9730 2500 50  0001 C CNN
 F 3 "~" H 9800 2500 50  0001 C CNN
 	1    9800 2500
@@
 F 0 "R23" H 9470 3346 50  0000 L CNN
 F 1 "1K" H 9470 3255 50  0000 L CNN
-F 2 "" V 9330 3300 50  0001 C CNN
+F 2 "Resistor_SMD:R_0805_2012Metric" V 9330 3300 50  0001 C CNN
 F 3 "~" H 9400 3300 50  0001 C CNN
 	1    9400 3300
@@
 F 0 "R27" H 9870 3346 50  0000 L CNN
 F 1 "1K" H 9870 3255 50  0000 L CNN
-F 2 "" V 9730 3300 50  0001 C CNN
+F 2 "Resistor_SMD:R_0805_2012Metric" V 9730 3300 50  0001 C CNN
 F 3 "~" H 9800 3300 50  0001 C CNN
 	1    9800 3300
@@
 L Connector:Screw_Terminal_01x02 J5
 U 1 1 5D863D99
-P 5200 2750
-F 0 "J5" H 5280 2742 50  0000 L CNN
-F 1 "PV(AC)" H 5280 2651 50  0000 L CNN
-F 2 "TerminalBlock:TerminalBlock_Wuerth_691311400102_P7.62mm" H 5200 2750 50  0001 C CNN
-F 3 "~" H 5200 2750 50  0001 C CNN
-	1    5200 2750
-	1    0    0    -1
+P 5200 2850
+F 0 "J5" H 5280 2842 50  0000 L CNN
+F 1 "PV(AC)" H 5280 2751 50  0000 L CNN
+F 2 "TerminalBlock:TerminalBlock_Wuerth_691311400102_P7.62mm" H 5200 2850 50  0001 C CNN
+F 3 "~" H 5200 2850 50  0001 C CNN
+	1    5200 2850
+	1    0    0    1
 $EndComp
 Text Label 7100 950  2    50   ~ 0
@@
 F 0 "R15" H 8170 2496 50  0000 L CNN
 F 1 "R" H 8170 2405 50  0000 L CNN
-F 2 "" V 8030 2450 50  0001 C CNN
+F 2 "Resistor_SMD:R_0805_2012Metric" V 8030 2450 50  0001 C CNN
 F 3 "~" H 8100 2450 50  0001 C CNN
 	1    8100 2450
@@
 L Connector:Conn_01x02_Female J7
 U 1 1 5DA5A031
-P 10900 2750
-F 0 "J7" H 10928 2726 50  0000 L CNN
-F 1 "PWD" H 10928 2635 50  0000 L CNN
-F 2 "Connector_PinSocket_2.54mm:PinSocket_1x02_P2.54mm_Vertical" H 10900 2750 50  0001 C CNN
-F 3 "~" H 10900 2750 50  0001 C CNN
-	1    10900 2750
-	1    0    0    -1
+P 10900 2850
+F 0 "J7" H 10928 2826 50  0000 L CNN
+F 1 "PWD" H 10928 2735 50  0000 L CNN
+F 2 "Connector_PinSocket_2.54mm:PinSocket_1x02_P2.54mm_Vertical" H 10900 2850 50  0001 C CNN
+F 3 "~" H 10900 2850 50  0001 C CNN
+	1    10900 2850
+	1    0    0    1
 $EndComp
 Wire Wire Line
@@
 F 0 "R16" V 8343 4600 50  0000 C CNN
 F 1 "R" V 8434 4600 50  0000 C CNN
-F 2 "" V 8480 4600 50  0001 C CNN
+F 2 "Resistor_SMD:R_0805_2012Metric" V 8480 4600 50  0001 C CNN
 F 3 "~" H 8550 4600 50  0001 C CNN
 	1    8550 4600
@@
 F 0 "R19" H 9120 6096 50  0000 L CNN
 F 1 "R" H 9120 6005 50  0000 L CNN
-F 2 "" V 8980 6050 50  0001 C CNN
+F 2 "Resistor_SMD:R_0805_2012Metric" V 8980 6050 50  0001 C CNN
 F 3 "~" H 9050 6050 50  0001 C CNN
 	1    9050 6050
@@
 F 0 "R18" H 8870 6096 50  0000 L CNN
 F 1 "R" H 8870 6005 50  0000 L CNN
-F 2 "" V 8730 6050 50  0001 C CNN
+F 2 "Resistor_SMD:R_0805_2012Metric" V 8730 6050 50  0001 C CNN
 F 3 "~" H 8800 6050 50  0001 C CNN
 	1    8800 6050
@@
 F 0 "R13" V 6300 3450 50  0000 L CNN
 F 1 "R" V 6300 3650 50  0000 L CNN
-F 2 "" V 6330 3600 50  0001 C CNN
+F 2 "Resistor_SMD:R_0805_2012Metric" V 6330 3600 50  0001 C CNN
 F 3 "~" H 6400 3600 50  0001 C CNN
 	1    6400 3600
@@
 F 0 "R28" H 6370 1346 50  0000 L CNN
 F 1 "1K" H 6370 1255 50  0000 L CNN
-F 2 "" V 6230 1300 50  0001 C CNN
+F 2 "Resistor_SMD:R_0805_2012Metric" V 6230 1300 50  0001 C CNN
 F 3 "~" H 6300 1300 50  0001 C CNN
 	1    6300 1300
@@
 F 0 "R29" H 6770 1346 50  0000 L CNN
 F 1 "1K" H 6770 1255 50  0000 L CNN
-F 2 "" V 6630 1300 50  0001 C CNN
+F 2 "Resistor_SMD:R_0805_2012Metric" V 6630 1300 50  0001 C CNN
 F 3 "~" H 6700 1300 50  0001 C CNN
 	1    6700 1300
@@
 F 0 "R14" V 7593 2300 50  0000 C CNN
 F 1 "R" V 7684 2300 50  0000 C CNN
-F 2 "" V 7730 2300 50  0001 C CNN
+F 2 "Resistor_SMD:R_0805_2012Metric" V 7730 2300 50  0001 C CNN
 F 3 "~" H 7800 2300 50  0001 C CNN
 	1    7800 2300
@@
 Wire Wire Line
 	1850 750  1850 850
+Wire Wire Line
+	2200 1400 2500 1400
+Wire Wire Line
+	2200 1400 2200 1500
+Wire Wire Line
+	2200 1400 2200 750
+Wire Wire Line
+	2200 750  1850 750
+Connection ~ 2200 1400
+Connection ~ 1850 750
 $EndSCHEMATC

Commit message: the new one 2/10/2019
Parts:
- IC1: symbol UImeasurement:TC1014-3.0VCT713 -> INVBackMeasurement-rescue:TC1014-3.0VCT713-UImeasurement
- IC2, IC3, IC4, IC5, IC6, IC7: symbol UImeasurement:HCPL-181-000E -> INVBackMeasurement-rescue:HCPL-181-000E-UImeasurement
- U1: symbol UImeasurement:MCP39F511 -> INVBackMeasurement-rescue:MCP39F511-UImeasurement
- U2: symbol dk_Current-Sensors:ACS712ELCTR-20A-T_NRND -> INVBackMeasurement-rescue:ACS712ELCTR-20A-T_NRND-dk_Current-Sensors
- U3: symbol UImeasurement:dsPIC33CK256MP502 -> INVBackMeasurement-rescue:dsPIC33CK256MP502-UImeasurement
Changed lines of the file:
@@
 	3300 1600 3800 1600
 $Comp
-L dk_Current-Sensors:ACS712ELCTR-20A-T_NRND U2
+L INVBackMeasurement-rescue:ACS712ELCTR-20A-T_NRND-dk_Current-Sensors U2
 U 1 1 5D857F1D
 P 2900 1500
@@
 	5100 1350 5100 1100
 $Comp
-L UImeasurement:HCPL-181-000E IC3
+L INVBackMeasurement-rescue:HCPL-181-000E-UImeasurement IC3
 U 1 1 5D8CB8DF
 P 9800 1000
@@
 	10800 1100 10600 1100
 $Comp
-L UImeasurement:HCPL-181-000E IC4
+L INVBackMeasurement-rescue:HCPL-181-000E-UImeasurement IC4
 U 1 1 5D9D6A8A
 P 9800 1900
@@
 	10800 2000 10600 2000
 $Comp
-L UImeasurement:HCPL-181-000E IC5
+L INVBackMeasurement-rescue:HCPL-181-000E-UImeasurement IC5
 U 1 1 5D9E47F4
 P 9800 2750
@@
 	9400 3050 9800 3050
 $Comp
-L UImeasurement:HCPL-181-000E IC6
+L INVBackMeasurement-rescue:HCPL-181-000E-UImeasurement IC6
 U 1 1 5D9F17CF
 P 9800 3550
@@
 $EndComp
 $Comp
-L UImeasurement:HCPL-181-000E IC2
+L INVBackMeasurement-rescue:HCPL-181-000E-UImeasurement IC2
 U 1 1 5DA334F6
 P 7550 2300
@@
 	8150 4600 8400 4600
 $Comp
-L UImeasurement:dsPIC33CK256MP502 U3
+L INVBackMeasurement-rescue:dsPIC33CK256MP502-UImeasurement U3
 U 1 1 5D87DD93
 P 7650 5000
@@
 3.3VDC
 $Comp
-L UImeasurement:TC1014-3.0VCT713 IC1
+L INVBackMeasurement-rescue:TC1014-3.0VCT713-UImeasurement IC1
 U 1 1 5DD378A4
 P 6650 3400
@@
 	1400 5000 1100 5000
 $Comp
-L UImeasurement:MCP39F511 U1
+L INVBackMeasurement-rescue:MCP39F511-UImeasurement U1
 U 1 1 5D878282
 P 2050 5250
@@
 AGND
 $Comp
-L UImeasurement:HCPL-181-000E IC7
+L INVBackMeasurement-rescue:HCPL-181-000E-UImeasurement IC7
 U 1 1 5D97412D
 P 6700 1550

Commit message: the new one
Parts:
- removed R12: 2m, InvertorMeasurement_kicad:ShuntMF0.0002Ohm2512, symbol Device:R_Shunt
- added J11: Screw_Terminal_01x02, TerminalBlock:TerminalBlock_Wuerth_691311400102_P7.62mm, symbol Connector:Screw_Terminal_01x02
- added R12: 2.49R, Resistor_SMD:R_0805_2012Metric, symbol Device:R
- added R33: CSNL2512FT2L00, InvertorMeasurement_kicad:ShuntMF0.0002Ohm2512, symbol UImeasurement:CSNL2512FT2L00
Connections:
- net AC\L: now also L2.2, R33.2
- net AC\L_OUT: now also L1.2, J11.1 (Pin_1), R33.1
- net AC\N: now also J11.2 (Pin_2)
- net at L1.1, R7.1: now also R12.1
- net at L2.1, R8.1: now also R12.2
Other:
- moved on the sheet: C3, C4
Changed lines of the file:
@@
 Wire Wire Line
 	4300 6000 4400 6000
-Wire Wire Line
-	4700 6000 4850 6000
 Text Label 1050 5400 0    50   ~ 0
 PT1
@@
 AC\L
 Wire Wire Line
-	5000 5500 5300 5500
-Wire Wire Line
-	5000 5900 5300 5900
-Wire Wire Line
-	4850 5400 4850 5600
-Wire Wire Line
-	4700 5400 4850 5400
-Wire Wire Line
-	4850 6000 4850 5800
-$Comp
-L Device:R_Shunt R12
-U 1 1 5DAD423A
-P 5000 5700
-F 0 "R12" H 4912 5654 50  0000 R CNN
-F 1 "2m" H 4912 5745 50  0000 R CNN
-F 2 "InvertorMeasurement_kicad:ShuntMF0.0002Ohm2512" V 4930 5700 50  0001 C CNN
-F 3 "~" H 5000 5700 50  0001 C CNN
-	1    5000 5700
-	-1   0    0    1
-$EndComp
+	4950 5300 5300 5500
+Wire Wire Line
+	4950 6100 5300 5900
 Connection ~ 3850 5700
 Wire Wire Line
@@
 L Device:C C3
 U 1 1 5E143A15
-P 1200 7200
-F 0 "C3" H 1315 7246 50  0000 L CNN
-F 1 "C" H 1315 7155 50  0000 L CNN
-F 2 "Capacitor_SMD:C_1206_3216Metric" H 1238 7050 50  0001 C CNN
-F 3 "~" H 1200 7200 50  0001 C CNN
-	1    1200 7200
+P 4500 3450
+F 0 "C3" H 4615 3496 50  0000 L CNN
+F 1 "C" H 4615 3405 50  0000 L CNN
+F 2 "Capacitor_SMD:C_1206_3216Metric" H 4538 3300 50  0001 C CNN
+F 3 "~" H 4500 3450 50  0001 C CNN
+	1    4500 3450
 	1    0    0    -1
 $EndComp
@@
 L Device:C C4
 U 1 1 5E144011
-P 1650 7200
-F 0 "C4" H 1765 7246 50  0000 L CNN
-F 1 "C" H 1765 7155 50  0000 L CNN
-F 2 "Capacitor_SMD:C_1206_3216Metric" H 1688 7050 50  0001 C CNN
-F 3 "~" H 1650 7200 50  0001 C CNN
-	1    1650 7200
+P 4950 3450
+F 0 "C4" H 5065 3496 50  0000 L CNN
+F 1 "C" H 5065 3405 50  0000 L CNN
+F 2 "Capacitor_SMD:C_1206_3216Metric" H 4988 3300 50  0001 C CNN
+F 3 "~" H 4950 3450 50  0001 C CNN
+	1    4950 3450
 	1    0    0    -1
 $EndComp
@@
 	6150 3400 6650 3400
 Wire Wire Line
-	1200 7350 1200 7600
-Wire Wire Line
-	1650 7350 1650 7600
-Wire Wire Line
-	1650 7050 1650 6900
-Text Label 1650 6900 0    50   ~ 0
+	4500 3600 4500 3850
+Wire Wire Line
+	4950 3600 4950 3850
+Wire Wire Line
+	4950 3300 4950 3150
+Text Label 4950 3150 0    50   ~ 0
 3.3VDC
-Text Label 1650 7600 0    50   ~ 0
+Text Label 4950 3850 0    50   ~ 0
 GNDD
 Text Label 3250 4100 0    50   ~ 0
@@
 AGND
 Wire Wire Line
-	1200 7050 1200 6900
-Text Label 1200 6900 0    50   ~ 0
+	4500 3300 4500 3150
+Text Label 4500 3150 0    50   ~ 0
 AVDD
-Text Label 1200 7600 0    50   ~ 0
+Text Label 4500 3850 0    50   ~ 0
 AGND
 $Comp
@@
 Connection ~ 2200 1400
 Connection ~ 1850 750
+Wire Wire Line
+	5250 4650 5250 4950
+Connection ~ 5250 4650
+Text Label 5250 4950 0    50   ~ 0
+AC\N_OUT
+$Comp
+L Connector:Screw_Terminal_01x02 J11
+U 1 1 5DABF6D1
+P 6000 4050
+F 0 "J11" H 6080 4042 50  0000 L CNN
+F 1 "Screw_Terminal_01x02" H 6080 3951 50  0000 L CNN
+F 2 "TerminalBlock:TerminalBlock_Wuerth_691311400102_P7.62mm" H 6000 4050 50  0001 C CNN
+F 3 "~" H 6000 4050 50  0001 C CNN
+	1    6000 4050
+	1    0    0    -1
+$EndComp
+Text Label 5400 4050 0    50   ~ 0
+AC\L_OUT
+Wire Wire Line
+	5400 4050 5800 4050
+Wire Wire Line
+	5400 4150 5800 4150
+Text Label 5400 4150 0    50   ~ 0
+AC\N_OUT
+$Comp
+L UImeasurement:CSNL2512FT2L00 R33
+U 1 1 5DBA8B14
+P 4950 5700
+F 0 "R33" V 4904 5805 50  0000 L CNN
+F 1 "CSNL2512FT2L00" V 4995 5805 50  0000 L CNN
+F 2 "InvertorMeasurement_kicad:ShuntMF0.0002Ohm2512" H 4950 5700 50  0001 L BNN
+F 3 "CSNL2512FT2L00" H 4950 5700 50  0001 L BNN
+F 4 "https://www.digikey.com/product-detail/en/stackpole-electronics-inc/CSNL2512FT2L00/CSNL2512FT2L00CT-ND/1646260?utm_source=snapeda&utm_medium=aggregator&utm_campaign=symbol" H 4950 5700 50  0001 L BNN "Field4"
+F 5 "2512 Stackpole Electronics" H 4950 5700 50  0001 L BNN "Field5"
+F 6 "Stackpole Electronics" H 4950 5700 50  0001 L BNN "Field6"
+F 7 "CSNL2512FT2L00CT-ND" H 4950 5700 50  0001 L BNN "Field7"
+F 8 "CSNL 2512 2 W 0.004O ±1% ±50 ppm/°C Metal Foil Current Sensing Chip Resistor" H 4950 5700 50  0001 L BNN "Field8"
+	1    4950 5700
+	0    1    1    0
+$EndComp
+Wire Wire Line
+	4700 5400 4950 5300
+Connection ~ 4950 5300
+Wire Wire Line
+	4700 6000 4950 6100
+Connection ~ 4950 6100
+$Comp
+L Device:R R12
+U 1 1 5DC8440C
+P 4400 5700
+F 0 "R12" H 4470 5746 50  0000 L CNN
+F 1 "2.49R" H 4470 5655 50  0000 L CNN
+F 2 "Resistor_SMD:R_0805_2012Metric" V 4330 5700 50  0001 C CNN
+F 3 "~" H 4400 5700 50  0001 C CNN
+	1    4400 5700
+	1    0    0    -1
+$EndComp
+Wire Wire Line
+	4400 5550 4400 5400
+Connection ~ 4400 5400
+Wire Wire Line
+	4400 5850 4400 6000
+Connection ~ 4400 6000
 $EndSCHEMATC

Commit message: 3/10/2019
Connections:
- net PWD is gone; now on net PWM: R22.1, R26.1
Changed lines of the file:
@@
 	9400 3150 8650 3150
 Text Label 8650 2350 0    50   ~ 0
-PWD
+PWM
 Wire Wire Line
 	9400 2350 8650 2350
